File: bench_board/bench_board.kicad_pcb (KiCad board)
At the start: 2 copper layers, 0 parts

Commit message: Bench board PCB layout: 4-layer stackup, placement, ground plane -- not routed, not DRC-clean (documented)
Synced 42 footprints from the finalized schematic. Added 2 inner
copper layers (4-layer total); In1.Cu is a dedicated GND plane per
the layout rules. 80x60mm outline -- generous, explicitly not whoop
dimensions, this board never flies.

Placement: force-directed auto-placement (suggest_placement) after
manually anchoring the MCU, IMU, power section, USB, and headers.
Verified 0 courtyard overlaps and 0 boundary violations before
applying. IMU sits ~41mm from the switching regulator, satisfying the
"don't place it near the switcher" rule -- computed from final
coordinates, not assumed.

Routing: no autorouter available (no Java, no freerouting.jar, no
Docker -- checked, not assumed). Manually routed the SPI bus and core
power chain as a real attempt, but direct point-to-point traces on the
MCU's 0.5mm-pitch LQFP pads produced actual short-circuit DRC errors
(SPI1_SCK shorting SPI1_MISO, etc) -- fine-pitch parts need real escape
routing, not straight lines. Deleted those traces rather than save a
board with hidden shorts. Board as committed has placement + ground
plane only; every net is still an unrouted airwire.

DRC: 106 violations remain (63 errors, 43 warnings), all
placement/footprint-driven now that the bad traces are gone. 60 of the
63 errors cluster at the USB-C connector's own fine pad pitch (0.15mm
actual vs 0.2mm board default) -- likely needs a relaxed clearance
rule for that footprint, not a placement fix; confirmed by re-running
DRC after a placement-margin change with no effect on the count.
Remaining 43 are cosmetic silkscreen overlaps from auto-placed field
text.

Full honest status, not just this summary: docs/bench-board-layout-status-2026-08-16.md.
No fab files produced -- layout reviewed here, not exported.
Parts:
- added C1: 10uF, Capacitor_SMD:C_0805_2012Metric, F.Cu at (17.9, 40.0)
- added C10: 100nF, Capacitor_SMD:C_0402_1005Metric, F.Cu at (44.9, 39.6)
- added C11: 2.2uF, Capacitor_SMD:C_0603_1608Metric, F.Cu at (25.6, 30.4)
- added C12: 2.2uF, Capacitor_SMD:C_0603_1608Metric, F.Cu at (24.5, 27.3)
- added C13: 1uF, Capacitor_SMD:C_0603_1608Metric, F.Cu at (37.8, 39.8)
- added C14: 10nF, Capacitor_SMD:C_0402_1005Metric, F.Cu at (44.9, 37.7)
- added C15: 4.7uF, Capacitor_SMD:C_0805_2012Metric, F.Cu at (48.5, 40.2)
- added C16: 100nF, Capacitor_SMD:C_0402_1005Metric, F.Cu at (47.7, 37.8)
- added C17: 10pF, Capacitor_SMD:C_0402_1005Metric, F.Cu at (33.1, 39.2)
- added C18: 10pF, Capacitor_SMD:C_0402_1005Metric, F.Cu at (33.2, 41.1)
- added C19: 100nF, Capacitor_SMD:C_0402_1005Metric, F.Cu at (44.7, 29.0)
- added C2: 22uF, Capacitor_SMD:C_0805_2012Metric, F.Cu at (25.4, 48.8)
- added C20: 100nF, Capacitor_SMD:C_0402_1005Metric, F.Cu at (45.1, 31.7)
- added C21: 100nF, Capacitor_SMD:C_0402_1005Metric, F.Cu at (46.1, 34.0)
- added C3: 2.2nF, Capacitor_SMD:C_0402_1005Metric, F.Cu at (14.4, 40.0)
- added C4: 10uF, Capacitor_SMD:C_0805_2012Metric, F.Cu at (26.0, 43.9)
- added C5: 22uF, Capacitor_SMD:C_0805_2012Metric, F.Cu at (45.1, 46.0)
- added C6: 100nF, Capacitor_SMD:C_0402_1005Metric, F.Cu at (45.0, 43.3)
- added C7: 100nF, Capacitor_SMD:C_0402_1005Metric, F.Cu at (45.2, 35.9)
- added C8: 100nF, Capacitor_SMD:C_0402_1005Metric, F.Cu at (44.9, 41.4)
- added C9: 100nF, Capacitor_SMD:C_0402_1005Metric, F.Cu at (38.6, 41.9)
- added J1: BATT_2S, Connector_PinHeader_2.54mm:PinHeader_1x02_P2.54mm_Vertical, F.Cu at (6.00, 30.0)
- added J2: BOOT0_JUMPER, Connector_PinHeader_2.54mm:PinHeader_1x02_P2.54mm_Vertical, F.Cu at (30.0, 12.0)
- added J3: USB-C, Connector_USB:USB_C_Receptacle_Amphenol_12401548E4-2A, F.Cu at (74.0, 30.0)
- added J4: CRSF_UART, Connector_PinHeader_2.54mm:PinHeader_1x04_P2.54mm_Vertical, F.Cu at (30.0, 47.0)
- added J5: DSHOT_M1-M4, Connector_PinHeader_2.54mm:PinHeader_1x05_P2.54mm_Vertical, F.Cu at (40.0, 47.0)
- added J6: SWD, Connector_PinHeader_2.54mm:PinHeader_1x05_P2.54mm_Vertical, F.Cu at (62.0, 47.0)
- added L1: 2.2uH, Inductor_SMD:L_1210_3225Metric, F.Cu at (20.0, 45.0)
- added R1: 40.2k, Resistor_SMD:R_0402_1005Metric, F.Cu at (22.3, 48.6)
- added R2: 7.32k, Resistor_SMD:R_0402_1005Metric, F.Cu at (27.0, 40.0)
- added R3: 10k, Resistor_SMD:R_0402_1005Metric, F.Cu at (48.4, 43.5)
- added R4: 10k, Resistor_SMD:R_0402_1005Metric, F.Cu at (26.6, 27.8)
- added R5: 22R, Resistor_SMD:R_0402_1005Metric, F.Cu at (53.5, 29.5)
- added R6: 22R, Resistor_SMD:R_0402_1005Metric, F.Cu at (53.5, 27.5)
- added R7: 5.1k, Resistor_SMD:R_0402_1005Metric, F.Cu at (56.5, 35.5)
- added R8: 5.1k, Resistor_SMD:R_0402_1005Metric, F.Cu at (56.5, 32.5)
- added U1: STM32F405RGT6, Package_QFP:LQFP-64_10x10mm_P0.5mm, F.Cu at (35.0, 30.0)
- added U2: TPS563201, Package_TO_SOT_SMD:SOT-23-6, F.Cu at (14.0, 45.0)
- added U3: AMS1117-3.3, Package_TO_SOT_SMD:SOT-223-3_TabPin2, F.Cu at (14.0, 52.0)
- added U4: MPU-6000, Sensor_Motion:InvenSense_QFN-24_4x4mm_P0.5mm, F.Cu at (48.0, 22.0)
- added U5: USBLC6-2SC6, Package_TO_SOT_SMD:SOT-23-6, F.Cu at (65.0, 24.0)
- added Y1: 8MHz, Crystal:Crystal_SMD_3225-4Pin_3.2x2.5mm, F.Cu at (26.0, 34.0)
Routing:
- added copper zone on In1.Cu, net GND
Other:
- board outline added: 80 x 60 mm
- copper layers 2 -> 4
