File: bench_board/bench_board.kicad_sch (KiCad schematic)
At the start: 45 parts, among them J1 BATT_4S, J2 BOOT0_JUMPER, J3 USB-C, J4 CRSF_UART, J5 DSHOT_M1-M4, J6 SWD, U1 STM32F405RGT6, U2 TPS54336ADDA, U4 MPU-6000, U5 USBLC6-2SC6, Y1 8MHz

Commit message: RX 5V rail (MT3608) + telemetry header into the schematic; ERC 0/0
Item 1 of the board-finalization batch. Executes both lead decisions.

RX POWER: MT3608 boost (LCSC C84817), 3.3V -> 5.0V, dedicated to the
receiver. Verified rather than assumed, on the same criteria that picked
the MPU-6000 and IST8310: native KiCad symbol exists
(Regulator_Switching:MT3608), part is orderable at JLCPCB (Extended, not
Basic -- setup fee applies), 162k in stock, $0.11 @1+.

INPUT SIDE IS 3.3V, AND THE DATASHEET DECIDES IT: the MT3608's absolute
maximum input is 24V, and this board is 6S-rated -- 6S peak is 25.2V.
Battery-side input would exceed the part's rating by 1.2V at full charge.
That is not a margin question. The 3.3V rail is also the quieter choice
(no second high-voltage switching node near the IMU), and the double-
conversion penalty is ~0.1W at 100mA, which is irrelevant here.

Recorded honestly in the doc: the lead decision cited "the industry-
standard whoop answer", but that research is for 1S whoops where the
battery is BELOW 5V. On a 4S/6S-rated board the same reasoning would
normally imply a buck. The conclusion still holds, for a different reason
than the one cited -- flagged so a future reader checking the whoop
reference does not conclude the part choice is wrong.

Feedback divider R12=73.2k / R13=10.0k gives 4.992V (FB ref 0.6V), within
0.2% of target on standard values. L2 reuses L1's exact value and
footprint (10uH 1210), one fewer distinct BOM line. D1 SS34 is mandatory,
not optional -- the MT3608 is non-synchronous.

RX DATA stays 3.3V logic on the existing CRSF nets; the receiver takes 5V
for power and 3.3V for signalling, the standard ELRS arrangement. Checked
against vendor documentation for the receiver CLASS, not the specific
unit -- no receiver is selected yet (David-only). The doc says plainly to
confirm the exact model's logic level before first power-on, and it is on
the runbook's Stage 7 checklist.

TELEMETRY: J8, 3-pin (TELEM_TX / GND / 3V3) on th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
Parts:
- added C25: 10uF 16V, Capacitor_SMD:C_0805_2012Metric, symbol Device:C
- added C26: 22uF 16V, Capacitor_SMD:C_0805_2012Metric, symbol Device:C
- added D1: SS34, Diode_SMD:D_SMA, symbol Device:D_Schottky
- added J7: RX_PWR_5V, Connector_PinHeader_2.54mm:PinHeader_1x02_P2.54mm_Vertical, symbol Connector:Conn_01x02_Pin
- added J8: TELEM_TX, Connector_PinHeader_2.54mm:PinHeader_1x03_P2.54mm_Vertical, symbol Connector:Conn_01x03_Pin
- added L2: 10uH, Inductor_SMD:L_1210_3225Metric, symbol Device:L
- added R12: 73.2k, Resistor_SMD:R_0603_1608Metric, symbol Device:R
- added R13: 10.0k, Resistor_SMD:R_0603_1608Metric, symbol Device:R
- added U6: MT3608, Package_TO_SOT_SMD:SOT-23-6, symbol Regulator_Switching:MT3608
Connections:
- net 3V3: now also C25.1, J8.3 (Pin_3), L2.1, U6.4 (EN), U6.5 (IN)
- net GND: now also C25.2, C26.2, J7.2 (Pin_2), J8.2 (Pin_2), R13.2, U6.2 (GND)
- net TELEM_TX: now reaches U1.51 (PC10)
- net TELEM_TX: now also J8.1 (Pin_1)
- new net 5V_RX: C26.1, D1.2 (A), J7.1 (Pin_1), R12.1
- new net BOOST_SW: D1.1 (K), L2.2, U6.1 (SW)
- new net VFB_5V: R12.2, R13.1, U6.3 (FB)
- no-connect marks 35 -> 34

Commit message: Collision-avoidance provisioning: audit found 2 real conflicts, both fixed
Item 2. Audited the expansion bus against the REAL pin budget and REAL
datasheets rather than from memory, and it did not pass as-specified --
two conflicts, both now resolved in the schematic.

CONFLICT 1: PC10 was double-allocated. stm32f405-pin-assignment.md gives
it to telemetry; expansion-bus-spec.md gives it to the bus as spare
UART_TX. Item 1 of this batch made the collision concrete by wiring the
telemetry header to it.

Resolved by splitting USART3 by DIRECTION, which works because both users
are unidirectional and opposite: PC10 TX to the ground station, PC11 RX
from the forward lidar. Full-duplex hardware, one shared baud register --
and both want 115200 anyway (the firmware's existing TELEM_BAUD and the
TF-Luna's factory default). Cost: the bus is now RX-only and cannot carry
a bidirectional companion link. Acceptable per the Build Plan (companion
computer is Stage 8; v1 tracking moves to a ground station), and the doc
names PA9 as the pin to revisit if that changes.

CONFLICT 2: the TF-Luna needs 5V +-0.1V and the expansion header carried
3.3V only -- as specified, the forward lidar could not be powered at all.
Resolved by adding 5V on expansion pin 13, fed from the MT3608 rail. Full
budget shown: ~170mA average total, ~300mA drawn from 3.3V after boost
losses, against a 3A supply. Flagged explicitly as a deliberate deviation
from the lead decision's "for the receiver alone" -- the decision's
PURPOSE was to kill the supply-voltage question with hardware, and the
lidar has the identical problem. Depopulating pin 13 reverts it if David
disagrees.

No I2C address conflict: IST8310 0x0E, VL53L1X 0x29, TF-Luna 0x10 (if run
in I2C mode) are all distinct. No mux needed -- the task permitted a mux
footprint and it turned out not to be required.

THE HONESTY THAT MATTERS MOST is the TF-Luna's 2-degree field of view: at
8m that cone is ~28cm across. It is a pencil beam. It will not see a d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
Parts:
- added J9: EXPANSION_BUS, Connector_PinHeader_2.54mm:PinHeader_1x14_P2.54mm_Vertical, symbol Connector:Conn_01x14_Pin
Connections:
- net 3V3: now also J9.1 (Pin_1)
- net 5V_RX: now also J9.13 (Pin_13)
- net GND: now also J9.14 (Pin_14), J9.2 (Pin_2)
- net EXP_IRQ1: now reaches U1.10 (PC2)
- net EXP_IRQ1: now also J9.11 (Pin_11)
- net EXP_IRQ2: now reaches U1.11 (PC3)
- net EXP_IRQ2: now also J9.12 (Pin_12)
- net EXP_I2C_SCL: now reaches U1.29 (PB10)
- net EXP_I2C_SCL: now also J9.3 (Pin_3)
- net EXP_I2C_SDA: now reaches U1.30 (PB11)
- net EXP_I2C_SDA: now also J9.4 (Pin_4)
- net EXP_SPI_SCK: now reaches U1.34 (PB13)
- net EXP_SPI_SCK: now also J9.5 (Pin_5)
- net EXP_SPI_MISO: now reaches U1.35 (PB14)
- net EXP_SPI_MISO: now also J9.7 (Pin_7)
- net EXP_SPI_MOSI: now reaches U1.36 (PB15)
- net EXP_SPI_MOSI: now also J9.6 (Pin_6)
- net EXP_UART_RX: now reaches U1.52 (PC11)
- net EXP_UART_RX: now also J9.10 (Pin_10)
- net EXP_SPI_CS1: now reaches U1.8 (PC0)
- net EXP_SPI_CS1: now also J9.8 (Pin_8)
- net EXP_SPI_CS2: now reaches U1.9 (PC1)
- net EXP_SPI_CS2: now also J9.9 (Pin_9)
- no-connect marks 34 -> 24
