File: bench_board/bench_board.kicad_sch (KiCad schematic)
At the start: 63 parts, among them J1 BATT_4S, J10 BUZZER, J2 BOOT0_JUMPER, J3 USB-C, J4 CRSF_UART, J5 DSHOT_M1-M4, J6 SWD, J7 RX_PWR_5V, J8 TELEM_TX, J9 EXPANSION_BUS, Q1 AO3400A, U1 STM32F405RGT6, U2 TPS54336ADDA, U4 MPU-6000, U5 USBLC6-2SC6, U6 MT3608, Y1 8MHz

Commit message: Item 3: crystal load caps C17/C18 10pF -> 33pF (CL=20pF crystal, manufacturer-confirmed)
Y1 (C115962, YXC X50328MSB2GI) is a 20pF-load crystal per the Yangxing
spec sheet read in the 2026-08-18 datasheet pass. 33pF gives
CL = 33/2 + ~3 stray = 19.5pF against the 20pF spec; the previous 10pF
pair ran the oscillator at ~8pF, ~+200-350ppm fast. Part: FH
0402CG330J500NT, LCSC C1562, C0G 50V, Basic library, 690k stock -- C0G
is also the right dielectric for load caps. Value-only change,
schematic and board together; ERC 0; guard PASS 53/2/95 unchanged.

C1 confirmed carried: schematic/board value still '10uF 50V X7S 1210'
(GCM32EC71H106KA03 / C126612 bias-verified resolution intact).

Co-Authored-By: Claude Fable 5 <noreply@anthropic.com>
Parts:
- C17, C18: value 10pF -> 33pF
Changed lines of the file:
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@@
 			)
 		)
-		(property "Value" "10pF"
+		(property "Value" "33pF"
 			(at 350.52 227.33 0)
 			(show_name no)
@@
 			)
 		)
-		(property "Value" "10pF"
+		(property "Value" "33pF"
 			(at 374.65 227.33 0)
 			(show_name no)

Commit message: Batch 7 review fixes: worst-case UVLO honesty, quantified via-in-pad, traceable specs
Independent review (fresh Opus agent): 0 BLOCKER, 1 HIGH, 4 MEDIUM,
6 LOW. It reproduced the EN divider arithmetic exactly (including a
worst-case 1% resistor sweep: EN 2.62V max at 25.2V -- violation
closed), traced C20's GND return copper to the plane via, verified
guard hashes hash-for-hash on all board commits, and accounted for
every copper delta -- zero scope creep. Acted on here:

- HIGH: the UVLO thresholds were computed from TYPICAL EN-comparator
  values; at datasheet LIMITS start = 12.0-13.0V and stop = 10.1-11.0V
  part-to-part (comparator tolerance dominates the resistors ~6x).
  Order sheet + README now state the ranges, raise the bench-supply
  instruction to >=13.5V (a worst-case part starts at ~12.95V), and
  say plainly this UVLO is brownout protection, NOT LiPo cell
  protection -- the firmware low-battery policy remains the pack
  guardian.
- MEDIUM: README gate line no longer claims 'every board commit
  carries a PASS' -- the item-1 commit carries a FAIL + same-commit
  re-baseline, now stated as such. R16.P2's via is called what it is
  (via-in-pad, 0.22mm of the 0.30mm drill inside the pad -- deepest on
  the board) in the fab remark. ORDER-SHEET's stale '93 parity' line
  fixed to 95. R16/R17/C20/C17/C18 now carry LCSC/Voltage/Tolerance/
  Dielectric properties in the schematic per project convention -- the
  50V rating and 1% tolerance live in the design source, not only in a
  hand-maintained CSV. ERC 0; guard PASS 53/2/95 unchanged.
- LOW: C11481 added to the verify-at-matching list with its alternate
  (C327365) -- its stock reads inconsistently across sources; stale
  stock notes refreshed; Y1's snapshot caveat closed (review confirmed
  live: Basic, 339k) and the review's oscillator gain-margin check
  (gm_crit 0.59mA/V vs 1mA/V limit) recorded in the BOM row.

Not changed, recorded: parity stays 95 (fully matching the new
footprint fields board-side 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
Parts:
- C17, C18: LCSC (none) -> C1562; Voltage (none) -> 50V
- C20: Dielectric (none) -> X7R; LCSC (none) -> C106861; Voltage (none) -> 50V
- R16: LCSC (none) -> C11481; Tolerance (none) -> 1%
- R17: LCSC (none) -> C25765; Tolerance (none) -> 1%
Changed lines of the file:
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@@
 			)
 		)
+    (property "LCSC" "C1562" (at 350.52 224.79 0)
+      (effects (font (size 1.27 1.27)) (hide yes))
+    )
+    (property "Voltage" "50V" (at 350.52 224.79 0)
+      (effects (font (size 1.27 1.27)) (hide yes))
+    )
 		(pin "1"
 		)
@@
 			)
 		)
+    (property "LCSC" "C1562" (at 374.65 224.79 0)
+      (effects (font (size 1.27 1.27)) (hide yes))
+    )
+    (property "Voltage" "50V" (at 374.65 224.79 0)
+      (effects (font (size 1.27 1.27)) (hide yes))
+    )
 		(pin "1"
 		)
@@
 			)
 		)
+    (property "LCSC" "C106861" (at 444.5 270.51 0)
+      (effects (font (size 1.27 1.27)) (hide yes))
+    )
+    (property "Voltage" "50V" (at 444.5 270.51 0)
+      (effects (font (size 1.27 1.27)) (hide yes))
+    )
+    (property "Dielectric" "X7R" (at 444.5 270.51 0)
+      (effects (font (size 1.27 1.27)) (hide yes))
+    )
 		(pin "1"
 		)
@@
 			)
 		)
+    (property "LCSC" "C11481" (at 381.0 35.56 0)
+      (effects (font (size 1.27 1.27)) (hide yes))
+    )
+    (property "Tolerance" "1%" (at 381.0 35.56 0)
+      (effects (font (size 1.27 1.27)) (hide yes))
+    )
 		(pin "1"
 		)
@@
 			)
 		)
+    (property "LCSC" "C25765" (at 381.0 49.53 0)
+      (effects (font (size 1.27 1.27)) (hide yes))
+    )
+    (property "Tolerance" "1%" (at 381.0 49.53 0)
+      (effects (font (size 1.27 1.27)) (hide yes))
+    )
 		(pin "1"
 		)
